File: hardware/EDA-Files/REG1-Front-Universal/REG1-Front-Universal_catia.kicad_pcb (KiCad board)
At the start: 2 copper layers, 25.4 x 52.8 mm, 12 parts, among them J1 Conn_02x04_Odd_Even, SW1 Prog, SW2 Func, SW3 Res, SW4 BL

Commit message: Front V00.02
Other:
- board size 25.4 x 52.8 mm -> 15.3 x 42.6 mm
- board text removed: "JLCJLCJLCJLC"
Changed lines of the file:
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@@
   (general
     (thickness 1.6)
-    (drawings 41)
+    (drawings 21)
     (tracks 113)
     (zones 0)
@@
     )
   )
-  (gr_arc (start 103.55 153) (end 103.55 154) (angle -180) (layer Edge.Cuts) (width 0.05))
-  (gr_line (start 96.6 154) (end 103.55 154) (layer Edge.Cuts) (width 0.05))
   (gr_line (start 103.55 152) (end 98.5 152) (layer Edge.Cuts) (width 0.05))
-  (gr_arc (start 108.35 153) (end 108.35 152) (angle -180) (layer Edge.Cuts) (width 0.05))
-  (gr_line (start 113.2 152) (end 108.35 152) (layer Edge.Cuts) (width 0.05))
-  (gr_line (start 108.35 154) (end 115.2 154) (layer Edge.Cuts) (width 0.05))
-  (gr_line (start 115.2 107.4) (end 108.25 107.4) (layer Edge.Cuts) (width 0.05))
-  (gr_line (start 108.25 109.4) (end 113.2 109.4) (layer Edge.Cuts) (width 0.05))
-  (gr_arc (start 108.25 108.4) (end 108.25 107.4) (angle -180) (layer Edge.Cuts) (width 0.05))
-  (gr_arc (start 103.45 108.4) (end 103.45 109.4) (angle -180) (layer Edge.Cuts) (width 0.05))
-  (gr_line (start 93.2 157.2) (end 93.2 104.4) (layer Edge.Cuts) (width 0.05))
-  (gr_line (start 118.6 157.2) (end 93.2 157.2) (layer Edge.Cuts) (width 0.05))
-  (gr_line (start 118.6 104.4) (end 118.6 157.2) (layer Edge.Cuts) (width 0.05))
-  (gr_line (start 93.2 104.4) (end 118.6 104.4) (layer Edge.Cuts) (width 0.05))
-  (gr_arc (start 96.6 153.6) (end 96.2 153.6) (angle -90) (layer Edge.Cuts) (width 0.05))
-  (gr_arc (start 115.2 153.6) (end 115.2 154) (angle -90) (layer Edge.Cuts) (width 0.05))
-  (gr_arc (start 96.6 107.8) (end 96.6 107.4) (angle -90) (layer Edge.Cuts) (width 0.05))
-  (gr_arc (start 115.2 107.8) (end 115.6 107.8) (angle -90) (layer Edge.Cuts) (width 0.05))
-  (gr_line (start 115.6 153.6) (end 115.6 107.8) (layer Edge.Cuts) (width 0.05))
-  (gr_line (start 96.2 153.6) (end 96.2 107.8) (layer Edge.Cuts) (width 0.05))
-  (gr_line (start 103.45 107.4) (end 96.6 107.4) (layer Edge.Cuts) (width 0.05))
-  (gr_text JLCJLCJLCJLC (at 105.75 105.95) (layer B.SilkS)
-    (effects (font (size 1 1) (thickness 0.15)) (justify mirror))
-  )
+  (gr_line (start 113.2 152) (end 103.55 152) (layer Edge.Cuts) (width 0.05))
   (gr_line (start 98.2 151.7) (end 98.5 152) (layer Edge.Cuts) (width 0.05))
   (gr_line (start 113.5 151.7) (end 113.2 152) (layer Edge.Cuts) (width 0.05))
@@
   (gr_line (start 98.2 151.7) (end 98.2 109.7) (layer Edge.Cuts) (width 0.05))
   (gr_line (start 113.5 109.7) (end 113.5 151.7) (layer Edge.Cuts) (width 0.05))
-  (gr_line (start 98.5 109.4) (end 103.45 109.4) (layer Edge.Cuts) (width 0.05))
+  (gr_line (start 98.5 109.4) (end 113.2 109.4) (layer Edge.Cuts) (width 0.05))
   (segment (start 100.625 118.425) (end 100.625 115.55) (width 0.2) (layer F.Cu) (net 1))
   (segment (start 100.65 140.125) (end 100.65 135.825) (width 0.2) (layer F.Cu) (net 1))
