File: hardware/EDA-Files/REG1-Front-Universal/REG1-Front-Universal.kicad_pcb (KiCad board)
At the start: 2 copper layers, 25.4 x 52.8 mm, 12 parts, among them J1 Conn_02x04_Odd_Even, SW1 Prog, SW2 Func, SW3 Res, SW4 BL

Commit message: REG1-Front-Universal V01.00
Parts:
- removed the G*** at (105.8, 146.4)
- removed the mouse-bite at (106.5, 151.8)
- removed the mouse-bite at (105.3, 109.5)
- added D3: Led2, LED_SMD:LED_0603_1608Metric, F.Cu at (59.0, 59.2)
- added D4: Led3, LED_SMD:LED_0603_1608Metric, F.Cu at (59.0, 65.0)
- added D5: Power, LED_SMD:LED_0603_1608Metric, F.Cu at (59.0, 83.0)
- added G***: LOGO, OpenKNX:OpenKNX_Logo_05x03, F.Cu at (48.7, 83.0)
- added G***: LOGO, OpenKNX:OpenKNX_Logo_07x05, B.Cu at (52.0, 50.6)
- added JP1: PowerLED Jumper, Jumper:SolderJumper-2_P1.3mm_Open_RoundedPad1.0x1.5mm, B.Cu at (60.3, 78.3)
- added R3: 2k2, Resistor_SMD:R_0402_1005Metric, F.Cu at (53.5, 73.3)
- added R4: 2k2, Resistor_SMD:R_0402_1005Metric, F.Cu at (56.0, 73.3)
- added R5: 2k2, Resistor_SMD:R_0402_1005Metric, F.Cu at (60.5, 79.0)
- added e: VAL**, DomsKiCADLib:mouse-bite-5.00mm-frame, F.Cu at (41.5, 43.3)
- added e: VAL**, DomsKiCADLib:mouse-bite-5.00mm-frame, F.Cu at (65.5, 43.3)
- added mouse-bite: mouse-bite-2.00mm-slot_1side, DomsKiCADLib:mouse-bite-2.00mm-slot_1side, F.Cu at (48.6, 86.2)
- added mouse-bite: VAL**, DomsKiCADLib:mouse-bite-5.00mm-frame, F.Cu at (41.5, 85.4)
- added mouse-bite: mouse-bite-2.00mm-slot_1side, DomsKiCADLib:mouse-bite-2.00mm-slot_1side, F.Cu at (59.4, 86.2)
- added mouse-bite: VAL**, DomsKiCADLib:mouse-bite-5.00mm-frame, F.Cu at (65.5, 85.4)
- added mouse-bite: mouse-bite-2.00mm-slot_1side, DomsKiCADLib:mouse-bite-2.00mm-slot_1side, F.Cu at (54.0, 42.4)
- D2: value Func -> Led1
- J1: value Conn_02x04_Odd_Even -> Frontpanel; footprint Connector_PinHeader_2.00mm:PinHeader_2x04_P2.00mm_Vertical_SMD -> EasyEDAModLib:C11050_FPC-SMD_P0.5-10P_LSXJ-H2.0-10P; moved to F.Cu
- R1, R2: value R -> 2k2
- SW1, SW3, SW4: footprint sirsydom:SW_Push_Xunpu_TS-1089S -> EasyEDAModLib:C455282_SW-SMD_4P-L4.2-W3.3-P2.15-LS5.1
- SW2: value Func -> Btn1; footprint sirsydom:SW_Push_Xunpu_TS-1089S -> EasyEDAModLib:C455282_SW-SMD_4P-L4.2-W3.3-P2.15-LS5.1
- moved D2 88.5 mm to (59.0, 53.0)
- moved D1 88.1 mm to (59.0, 47.0)
- moved SW2 88.0 mm to (50.0, 53.0), turned to 0 degrees
- moved SW1 87.6 mm to (50.0, 47.0), turned to 0 degrees
- moved SW4 84.6 mm to (50.0, 71.0), turned to 0 degrees
- moved R2 81.6 mm to (49.4, 73.3)
- moved R1 75.6 mm to (54.2, 70.6), turned to -90 degrees
- moved SW3 74.7 mm to (58.0, 71.0), turned to 0 degrees
- moved J1 71.0 mm to (54.0, 76.1), turned to 180 degrees
Connections:
- D1 pad 1: Net-(D1-Pad1) -> GND
- D1 pad 2: PROGLED -> Net-(D1-A)
- D2 pad 1: Net-(D2-Pad1) -> GND
- D2 pad 2: GPIO03 -> Net-(D2-A)
- J1 pad 1: GND -> GPIO23
- J1 pad 2: +3V3 -> RUN
- J1 pad 3: PROGLED -> GPIO25
- J1 pad 4: GPIO24 -> GPIO22
- J1 pad 5: GPIO03 -> GND
- J1 pad 6: RUN -> +3.3V
- J1 pad 7: PROGBTN -> GPIO24
- J1 pad 8: BOOTSEL_F -> GPIO7
- R1 pad 1: GND -> Net-(D1-A)
- R1 pad 2: Net-(D1-Pad1) -> GPIO25
- R2 pad 1: GND -> Net-(D2-A)
- R2 pad 2: Net-(D2-Pad1) -> GPIO6
- SW1 pad 1: PROGBTN -> GPIO23
- SW2 pad 1: GPIO24 -> GPIO7
- SW4 pad 1: BOOTSEL_F -> BOOTSEL
Routing:
- net GND: track 70.5 -> 121.4 mm, vias 6 -> 10
- net GPIO23: track 0.00 -> 44.0 mm, vias 0 -> 2
- net GPIO7: track 0.00 -> 35.3 mm, vias 0 -> 2
- net Net-(D1-A): track 0.00 -> 34.9 mm, vias 0 -> 2
- net BOOTSEL_F: track 28.0 -> 0.00 mm, vias 1 -> 0
- net Net-(D2-A): track 0.00 -> 27.4 mm, vias 0 -> 2
- net PROGLED: track 19.5 -> 0.00 mm, vias 1 -> 0
- net Net-(D3-A): track 0.00 -> 19.5 mm, vias 0 -> 2
- net PROGBTN: track 15.1 -> 0.00 mm, vias 1 -> 0
- net Net-(D4-A): track 0.00 -> 14.1 mm, vias 0 -> 2
- net +3.3V: track 0.00 -> 12.5 mm, vias 0 -> 1
- net BOOTSEL: track 0.00 -> 10.9 mm
- net GPIO03: track 9.26 -> 0.00 mm, vias 1 -> 0
- net GPIO25: track 0.00 -> 9.23 mm, vias 0 -> 2
- net GPIO24: track 10.1 -> 2.20 mm, vias 1 -> 0
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Other:
- board size 25.4 x 52.8 mm -> 28.5 x 52.8 mm
- net class Default removed
- rule pad_to_mask_clearance: 0.051 -> 0.038
- board text added: "REG1-Front-Universal V01.00 (c) Ing-Dom, 2023"
- board text removed: "3V3"
- board text removed: "BL"
- board text removed: "GND"
- board text removed: "GP24"
- board text removed: "GP3"
- board text removed: "PBTN"
- board text removed: "PLED"
- board text removed: "Prog"
- board text removed: "REG1-Front-Universal V00.02 © Ing-Dom, 2022"
- board text removed: "RES"
- board text removed: "Reset"

Commit message: increased size of Front-Universal, WIP
Parts:
- moved mouse-bite 0.10 mm to (54.0, 42.3)
- moved mouse-bite 0.10 mm to (48.6, 86.3)
- moved mouse-bite 0.10 mm to (59.4, 86.3)
Other:
- outline, holes or cut-outs redrawn
Changed lines of the file:
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@@
   )
   (footprint "DomsKiCADLib:mouse-bite-2.00mm-slot_1side" (layer "F.Cu")
-    (at 48.6 86.2)
+    (at 48.6 86.3)
     (attr through_hole board_only exclude_from_pos_files exclude_from_bom)
     (fp_text reference "mouse-bite" (at 0.2 2.5) (layer "F.SilkS") hide
@@
   )
   (footprint "DomsKiCADLib:mouse-bite-2.00mm-slot_1side" (layer "F.Cu")
-    (at 59.4 86.2)
+    (at 59.4 86.3)
     (attr through_hole board_only exclude_from_pos_files exclude_from_bom)
     (fp_text reference "mouse-bite" (at 0.4 2.8) (layer "F.SilkS") hide
@@
   )
   (footprint "DomsKiCADLib:mouse-bite-2.00mm-slot_1side" (layer "F.Cu")
-    (at 54 42.4 180)
+    (at 54 42.3 180)
     (attr through_hole board_only exclude_from_pos_files exclude_from_bom)
     (fp_text reference "mouse-bite" (at 0.2 2.2) (layer "F.SilkS") hide
@@
   (gr_line (start 45 71) (end 73.25 71)
     (stroke (width 0.1) (type default)) (layer "Eco1.User"))
-  (gr_line (start 46.35 85.3) (end 46.35 43.3)
+  (gr_line (start 46.15 85.3) (end 46.15 43.3)
     (stroke (width 0.05) (type solid)) (layer "Edge.Cuts"))
   (gr_line (start 63.25 41) (end 55.5 41)
@@
   (gr_line (start 56.5 87.6) (end 57.9 87.6)
     (stroke (width 0.05) (type solid)) (layer "Edge.Cuts"))
-  (gr_line (start 61.35 85.6) (end 60.9 85.6)
+  (gr_line (start 61.45 85.7) (end 60.9 85.7)
     (stroke (width 0.05) (type solid)) (layer "Edge.Cuts"))
-  (gr_line (start 51 85.6) (end 50.1 85.6)
+  (gr_line (start 51 85.7) (end 50.1 85.7)
     (stroke (width 0.05) (type solid)) (layer "Edge.Cuts"))
   (gr_line (start 50.1 87.6) (end 56.5 87.6)
     (stroke (width 0.05) (type solid)) (layer "Edge.Cuts"))
-  (gr_arc (start 52.8 42.7) (mid 52.712132 42.912132) (end 52.5 43)
+  (gr_arc (start 52.8 42.6) (mid 52.712132 42.812132) (end 52.5 42.9)
     (stroke (width 0.05) (type default)) (layer "Edge.Cuts"))
-  (gr_line (start 61.35 43) (end 55.5 43)
+  (gr_line (start 61.45 42.9) (end 55.5 42.9)
     (stroke (width 0.05) (type default)) (layer "Edge.Cuts"))
-  (gr_line (start 46.65 43) (end 46.35 43.3)
+  (gr_line (start 46.55 42.9) (end 46.15 43.3)
     (stroke (width 0.05) (type solid)) (layer "Edge.Cuts"))
-  (gr_arc (start 47.1 85.6) (mid 47.312132 85.687868) (end 47.4 85.9)
+  (gr_arc (start 47.1 85.7) (mid 47.312132 85.787868) (end 47.4 86)
     (stroke (width 0.05) (type default)) (layer "Edge.Cuts"))
-  (gr_line (start 61.65 85.3) (end 61.35 85.6)
+  (gr_line (start 61.85 85.3) (end 61.45 85.7)
     (stroke (width 0.05) (type solid)) (layer "Edge.Cuts"))
   (gr_arc (start 52.5 41) (mid 52.712132 41.087868) (end 52.8 41.3)
@@
   (gr_arc (start 63.25 41) (mid 63.532843 41.117157) (end 63.65 41.4)
     (stroke (width 0.05) (type default)) (layer "Edge.Cuts"))
-  (gr_line (start 46.65 85.6) (end 46.35 85.3)
+  (gr_line (start 46.55 85.7) (end 46.15 85.3)
     (stroke (width 0.05) (type default)) (layer "Edge.Cuts"))
   (gr_line (start 51.25 80.6) (end 56.75 80.6)
@@
   (gr_arc (start 60.9 87.6) (mid 60.687868 87.512132) (end 60.6 87.3)
     (stroke (width 0.05) (type default)) (layer "Edge.Cuts"))
-  (gr_arc (start 49.8 85.9) (mid 49.887868 85.687868) (end 50.1 85.6)
+  (gr_arc (start 49.8 86) (mid 49.887868 85.787868) (end 50.1 85.7)
     (stroke (width 0.05) (type default)) (layer "Edge.Cuts"))
   (gr_arc (start 63.65 87.2) (mid 63.532843 87.482843) (end 63.25 87.6)
     (stroke (width 0.05) (type default)) (layer "Edge.Cuts"))
-  (gr_arc (start 55.5 43) (mid 55.287868 42.912132) (end 55.2 42.7)
+  (gr_arc (start 55.5 42.9) (mid 55.287868 42.812132) (end 55.2 42.6)
     (stroke (width 0.05) (type default)) (layer "Edge.Cuts"))
-  (gr_line (start 61.65 43.3) (end 61.65 85.3)
+  (gr_line (start 61.85 43.3) (end 61.85 85.3)
     (stroke (width 0.05) (type solid)) (layer "Edge.Cuts"))
-  (gr_line (start 51 85.6) (end 51 80.85)
+  (gr_line (start 51 85.7) (end 51 80.85)
     (stroke (width 0.05) (type default)) (layer "Edge.Cuts"))
-  (gr_line (start 60.6 85.9) (end 60.6 87.3)
+  (gr_line (start 60.6 86) (end 60.6 87.3)
     (stroke (width 0.05) (type default)) (layer "Edge.Cuts"))
-  (gr_line (start 57.9 85.6) (end 57 85.6)
+  (gr_line (start 57.9 85.7) (end 57 85.7)
     (stroke (width 0.05) (type default)) (layer "Edge.Cuts"))
-  (gr_line (start 58.2 87.3) (end 58.2 85.9)
+  (gr_line (start 58.2 87.3) (end 58.2 86)
     (stroke (width 0.05) (type default)) (layer "Edge.Cuts"))
   (gr_arc (start 58.2 87.3) (mid 58.112132 87.512132) (end 57.9 87.6)
@@
   (gr_line (start 52.5 41) (end 44.75 41)
     (stroke (width 0.05) (type solid)) (layer "Edge.Cuts"))
-  (gr_line (start 46.65 43) (end 52.5 43)
+  (gr_line (start 46.55 42.9) (end 52.5 42.9)
     (stroke (width 0.05) (type solid)) (layer "Edge.Cuts"))
-  (gr_line (start 57 80.85) (end 57 85.6)
+  (gr_line (start 57 80.85) (end 57 85.7)
     (stroke (width 0.05) (type default)) (layer "Edge.Cuts"))
-  (gr_line (start 52.8 42.7) (end 52.8 41.3)
+  (gr_line (start 52.8 42.6) (end 52.8 41.3)
     (stroke (width 0.05) (type default)) (layer "Edge.Cuts"))
-  (gr_arc (start 60.6 85.9) (mid 60.687868 85.687868) (end 60.9 85.6)
+  (gr_arc (start 60.6 86) (mid 60.687868 85.787868) (end 60.9 85.7)
     (stroke (width 0.05) (type default)) (layer "Edge.Cuts"))
-  (gr_line (start 47.4 87.3) (end 47.4 85.9)
+  (gr_line (start 47.4 87.3) (end 47.4 86)
     (stroke (width 0.05) (type default)) (layer "Edge.Cuts"))
-  (gr_line (start 49.8 85.9) (end 49.8 87.3)
+  (gr_line (start 49.8 86) (end 49.8 87.3)
     (stroke (width 0.05) (type default)) (layer "Edge.Cuts"))
-  (gr_line (start 47.1 85.6) (end 46.65 85.6)
+  (gr_line (start 47.1 85.7) (end 46.55 85.7)
     (stroke (width 0.05) (type solid)) (layer "Edge.Cuts"))
   (gr_line (start 60.9 87.6) (end 63.25 87.6)
@@
   (gr_line (start 63.65 87.2) (end 63.65 41.4)
     (stroke (width 0.05) (type solid)) (layer "Edge.Cuts"))
-  (gr_line (start 61.35 43) (end 61.65 43.3)
+  (gr_line (start 61.45 42.9) (end 61.85 43.3)
     (stroke (width 0.05) (type default)) (layer "Edge.Cuts"))
-  (gr_arc (start 57.9 85.6) (mid 58.112132 85.687868) (end 58.2 85.9)
+  (gr_arc (start 57.9 85.7) (mid 58.112132 85.787868) (end 58.2 86)
     (stroke (width 0.05) (type default)) (layer "Edge.Cuts"))
   (gr_line (start 44.35 87.2) (end 44.35 41.4)
     (stroke (width 0.05) (type solid)) (layer "Edge.Cuts"))
-  (gr_line (start 55.2 41.3) (end 55.2 42.7)
+  (gr_line (start 55.2 41.3) (end 55.2 42.6)
     (stroke (width 0.05) (type default)) (layer "Edge.Cuts"))
   (gr_arc (start 44.75 87.6) (mid 44.467157 87.482843) (end 44.35 87.2)

Commit message: REG1-Front-Universal_V01.01
Parts:
- removed G***: LOGO, OpenKNX:OpenKNX_Logo_05x03
- removed G***: LOGO, OpenKNX:OpenKNX_Logo_07x05
- removed e (x2), mouse-bite (x2): VAL**, DomsKiCADLib:mouse-bite-5.00mm-frame
- removed mouse-bite (x3): mouse-bite-2.00mm-slot_1side, DomsKiCADLib:mouse-bite-2.00mm-slot_1side
- added G1: LOGO, OpenKNX:OpenKNX_Logo_10x10, B.Cu at (49.3, 62.6)
- added G2: LOGO, OpenKNX:CC-BY-NY-SA_12x4, B.Cu at (49.5, 73.4)
Routing:
- net GND: track 121.4 -> 136.3 mm, vias 10 -> 11
- net Net-(D1-A): track 34.9 -> 37.2 mm
- net BOOTSEL: track 10.9 -> 12.8 mm
Other:
- board size 28.5 x 52.8 mm -> 15.7 x 42.8 mm
- board text added: "REG1-Front-Universal V01.00a by Ing-Dom, 2025"
- board text removed: "JLCJLCJLCJLC"
- board text removed: "REG1-Front-Universal V01.00 (c) Ing-Dom, 2023"
