File: hardware/EDA-Files/REG1-Front-Universal/REG1-Front-Universal.kicad_sch (KiCad schematic)
At the start: 16 parts, among them J102 Frontpanel, SW1 Prog, SW2 Btn1, SW3 Res, SW4 BL

Commit message: REG1-Front-Universal_V01.01
Parts:
- D1: LCSC C2286 -> (none)
- D2, D3, D4, D5: LCSC C72043 -> (none)
- J102: LCSC C11050 -> (none)
- R1, R2, R3, R4, R5: LCSC C25879 -> (none)
- SW1, SW2, SW3, SW4: LCSC C455282 -> (none)
