File: hardware/EDA-Files/REG1-App-Universal/REG1-App-Universal.sch (KiCad schematic (older format))
At the start: 14 parts, among them J1 Conn_01x06, J10 Conn_01x22, J11 Conn_01x22, J12 Conn_01x22, J13 Conn_01x22, J14 Conn_01x22, J2 Conn_01x06, J3 Conn_01x10, J4 Conn_01x06, J5 Conn_01x10, J6 Conn_01x06, J7 Conn_01x22, J8 Conn_01x22, J9 Conn_01x22

Commit message: editorial V00.10 of App-Universal
Parts:
- removed J14: Conn_01x22, Connector_PinHeader_2.54mm:PinHeader_1x22_P2.54mm_Vertical, symbol Connector_Generic:Conn_01x22
- removed J5: Conn_01x10, Connector_PinHeader_2.54mm:PinHeader_1x10_P2.54mm_Vertical, symbol Connector_Generic:Conn_01x10
- added J1: REG1_App_Connector, Connector_PinHeader_2.54mm:PinHeader_1x10_P2.54mm_Horizontal, symbol OpenKNX:REG1_App_Connector
- J2: renamed from J3; footprint Connector_PinHeader_2.54mm:PinHeader_1x10_P2.54mm_Horizontal -> Connector_PinHeader_2.54mm:PinHeader_1x10_P2.54mm_Vertical
- renumbered J1 to J10, J4 to J11, J2 to J20, J6 to J21, J7 to J30, J8 to J31, J9 to J32, J10 to J33, J11 to J34, J12 to J35, J13 to J36
Connections:
- net at J2.1 (Pin_1): now also J1.1 (GP16)
- net at J2.10 (Pin_10): now also J1.10 (VCC2)
- net at J2.2 (Pin_2): now also J1.2 (GP17)
- net at J2.3 (Pin_3): now also J1.3 (GP18)
- net at J2.4 (Pin_4): now also J1.4 (GP26)
- net at J2.5 (Pin_5): now also J1.5 (GP27)
- net at J2.6 (Pin_6): now also J1.6 (GP28)
- net at J2.7 (Pin_7): now also J1.7 (GP29)
- net at J2.8 (Pin_8): now also J1.8 (GND)
- net at J2.9 (Pin_9): now also J1.9 (3V3)
Changed lines of the file:
@@
 Sheet 1 1
 Title "REG1-App-Universal"
-Date "2022-11-05"
-Rev "V00.02"
+Date "2023-01-31"
+Rev "V00.10"
 Comp "OpenKNX"
 Comment1 "by Ing-Dom <dom@ing-dom.de>"
@@
 $EndDescr
 $Comp
-L Connector_Generic:Conn_01x06 J1
+L Connector_Generic:Conn_01x06 J10
 U 1 1 635039A7
 P 5750 1650
-F 0 "J1" H 5830 1642 50  0000 L CNN
+F 0 "J10" H 5830 1642 50  0000 L CNN
 F 1 "Conn_01x06" H 5830 1551 50  0000 L CNN
 F 2 "Connector_Phoenix_MC:PhoenixContact_MC_1,5_6-G-3.5_1x06_P3.50mm_Horizontal" H 5750 1650 50  0001 C CNN
@@
 $EndComp
 $Comp
-L Connector_Generic:Conn_01x06 J2
+L Connector_Generic:Conn_01x06 J20
 U 1 1 6350429B
 P 5750 2350
-F 0 "J2" H 5830 2342 50  0000 L CNN
+F 0 "J20" H 5830 2342 50  0000 L CNN
 F 1 "Conn_01x06" H 5830 2251 50  0000 L CNN
 F 2 "Connector_Phoenix_MC:PhoenixContact_MC_1,5_6-G-3.5_1x06_P3.50mm_Horizontal" H 5750 2350 50  0001 C CNN
@@
 $EndComp
 $Comp
-L Connector_Generic:Conn_01x10 J3
+L Connector_Generic:Conn_01x10 J2
 U 1 1 63504940
 P 3950 2000
-F 0 "J3" H 4030 1992 50  0000 L CNN
+F 0 "J2" H 4030 1992 50  0000 L CNN
 F 1 "Conn_01x10" H 4030 1901 50  0000 L CNN
-F 2 "Connector_PinHeader_2.54mm:PinHeader_1x10_P2.54mm_Horizontal" H 3950 2000 50  0001 C CNN
+F 2 "Connector_PinHeader_2.54mm:PinHeader_1x10_P2.54mm_Vertical" H 3950 2000 50  0001 C CNN
 F 3 "~" H 3950 2000 50  0001 C CNN
 	1    3950 2000
@@
 $EndComp
 $Comp
-L Connector_Generic:Conn_01x10 J5
-U 1 1 6350840D
-P 3250 2000
-F 0 "J5" H 3168 2617 50  0000 C CNN
-F 1 "Conn_01x10" H 3168 2526 50  0000 C CNN
-F 2 "Connector_PinHeader_2.54mm:PinHeader_1x10_P2.54mm_Vertical" H 3250 2000 50  0001 C CNN
-F 3 "~" H 3250 2000 50  0001 C CNN
-	1    3250 2000
-	-1   0    0    -1
-$EndComp
-$Comp
-L Connector_Generic:Conn_01x06 J4
+L Connector_Generic:Conn_01x06 J11
 U 1 1 6350992D
 P 5200 1650
-F 0 "J4" H 5280 1642 50  0000 L CNN
+F 0 "J11" H 5280 1642 50  0000 L CNN
 F 1 "Conn_01x06" H 5280 1551 50  0000 L CNN
 F 2 "Connector_PinHeader_2.54mm:PinHeader_1x06_P2.54mm_Vertical" H 5200 1650 50  0001 C CNN
@@
 $EndComp
 $Comp
-L Connector_Generic:Conn_01x06 J6
+L Connector_Generic:Conn_01x06 J21
 U 1 1 6350ABDC
 P 5200 2350
-F 0 "J6" H 5280 2342 50  0000 L CNN
+F 0 "J21" H 5280 2342 50  0000 L CNN
 F 1 "Conn_01x06" H 5280 2251 50  0000 L CNN
 F 2 "Connector_PinHeader_2.54mm:PinHeader_1x06_P2.54mm_Vertical" H 5200 2350 50  0001 C CNN
@@
 	3450 2500 3750 2500
 $Comp
-L Connector_Generic:Conn_01x22 J7
+L Connector_Generic:Conn_01x22 J30
 U 1 1 63510167
 P 7250 2250
-F 0 "J7" H 7330 2242 50  0000 L CNN
+F 0 "J30" H 7330 2242 50  0000 L CNN
 F 1 "Conn_01x22" H 7330 2151 50  0000 L CNN
 F 2 "Connector_PinHeader_2.54mm:PinHeader_1x22_P2.54mm_Vertical" H 7250 2250 50  0001 C CNN
@@
 $EndComp
 $Comp
-L Connector_Generic:Conn_01x22 J8
+L Connector_Generic:Conn_01x22 J31
 U 1 1 63512B13
 P 7650 2250
-F 0 "J8" H 7730 2242 50  0000 L CNN
+F 0 "J31" H 7730 2242 50  0000 L CNN
 F 1 "Conn_01x22" H 7730 2151 50  0000 L CNN
 F 2 "Connector_PinHeader_2.54mm:PinHeader_1x22_P2.54mm_Vertical" H 7650 2250 50  0001 C CNN
@@
 $EndComp
 $Comp
-L Connector_Generic:Conn_01x22 J9
+L Connector_Generic:Conn_01x22 J32
 U 1 1 6351419E
 P 8100 2250
-F 0 "J9" H 8180 2242 50  0000 L CNN
+F 0 "J32" H 8180 2242 50  0000 L CNN
 F 1 "Conn_01x22" H 8180 2151 50  0000 L CNN
 F 2 "Connector_PinHeader_2.54mm:PinHeader_1x22_P2.54mm_Vertical" H 8100 2250 50  0001 C CNN
@@
 $EndComp
 $Comp
-L Connector_Generic:Conn_01x22 J10
+L Connector_Generic:Conn_01x22 J33
 U 1 1 635149EC
 P 8550 2250
-F 0 "J10" H 8630 2242 50  0000 L CNN
+F 0 "J33" H 8630 2242 50  0000 L CNN
 F 1 "Conn_01x22" H 8630 2151 50  0000 L CNN
 F 2 "Connector_PinHeader_2.54mm:PinHeader_1x22_P2.54mm_Vertical" H 8550 2250 50  0001 C CNN
@@
 $EndComp
 $Comp
-L Connector_Generic:Conn_01x22 J11
+L Connector_Generic:Conn_01x22 J34
 U 1 1 63515159
 P 9000 2250
-F 0 "J11" H 9080 2242 50  0000 L CNN
+F 0 "J34" H 9080 2242 50  0000 L CNN
 F 1 "Conn_01x22" H 9080 2151 50  0000 L CNN
 F 2 "Connector_PinHeader_2.54mm:PinHeader_1x22_P2.54mm_Vertical" H 9000 2250 50  0001 C CNN
@@
 $EndComp
 $Comp
-L Connector_Generic:Conn_01x22 J12
+L Connector_Generic:Conn_01x22 J35
 U 1 1 635157E5
 P 9350 2250
-F 0 "J12" H 9430 2242 50  0000 L CNN
+F 0 "J35" H 9430 2242 50  0000 L CNN
 F 1 "Conn_01x22" H 9430 2151 50  0000 L CNN
 F 2 "Connector_PinHeader_2.54mm:PinHeader_1x22_P2.54mm_Vertical" H 9350 2250 50  0001 C CNN
@@
 $EndComp
 $Comp
-L Connector_Generic:Conn_01x22 J13
+L Connector_Generic:Conn_01x22 J36
 U 1 1 6351EF69
 P 9800 2250
-F 0 "J13" H 9880 2242 50  0000 L CNN
+F 0 "J36" H 9880 2242 50  0000 L CNN
 F 1 "Conn_01x22" H 9880 2151 50  0000 L CNN
 F 2 "Connector_PinHeader_2.54mm:PinHeader_1x22_P2.54mm_Vertical" H 9800 2250 50  0001 C CNN
@@
 $EndComp
 $Comp
-L Connector_Generic:Conn_01x22 J14
-U 1 1 6351FD61
-P 10250 2250
-F 0 "J14" H 10330 2242 50  0000 L CNN
-F 1 "Conn_01x22" H 10330 2151 50  0000 L CNN
-F 2 "Connector_PinHeader_2.54mm:PinHeader_1x22_P2.54mm_Vertical" H 10250 2250 50  0001 C CNN
-F 3 "~" H 10250 2250 50  0001 C CNN
-	1    10250 2250
+L OpenKNX:REG1_App_Connector J1
+U 1 1 63D94379
+P 2850 2050
+F 0 "J1" H 2183 2725 50  0000 C CNN
+F 1 "REG1_App_Connector" H 2183 2634 50  0000 C CNN
+F 2 "Connector_PinHeader_2.54mm:PinHeader_1x10_P2.54mm_Horizontal" H 2850 2050 50  0001 C CNN
+F 3 "" H 2850 2050 50  0001 C CNN
+	1    2850 2050
 	1    0    0    -1
 $EndComp
