File: hardware/EDA-Files/REG1-App-8xDI/REG1-App-8xBE.kicad_sch (KiCad schematic)
At the start: 3 parts, among them J1 REG1_App_Connector, J10 Conn_01x08, J20 Conn_01x08

Commit message: wip 8xBE
Parts:
- J10, J20: footprint EasyEDALib:C2927509_CONN-TH_8P-P2.54_DIBO_DB2ERC-2.54-8P-GN -> EasyEDALib:CONN-TH_8P-P2.54_DIBO_DB2ERC-2.54-8P-GN; LCSC (none) -> C2927509
Changed lines of the file:
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@@
       (effects (font (size 1.27 1.27)) (justify left))
     )
-    (property "Footprint" "EasyEDALib:C2927509_CONN-TH_8P-P2.54_DIBO_DB2ERC-2.54-8P-GN" (at 83.82 77.47 0)
+    (property "Footprint" "EasyEDALib:CONN-TH_8P-P2.54_DIBO_DB2ERC-2.54-8P-GN" (at 83.82 77.47 0)
       (effects (font (size 1.27 1.27)) hide)
     )
     (property "Datasheet" "~" (at 83.82 77.47 0)
+      (effects (font (size 1.27 1.27)) hide)
+    )
+    (property "LCSC" "C2927509" (at 83.82 77.47 0)
       (effects (font (size 1.27 1.27)) hide)
     )
@@
       (effects (font (size 1.27 1.27)) (justify left))
     )
-    (property "Footprint" "EasyEDALib:C2927509_CONN-TH_8P-P2.54_DIBO_DB2ERC-2.54-8P-GN" (at 83.82 102.87 0)
+    (property "Footprint" "EasyEDALib:CONN-TH_8P-P2.54_DIBO_DB2ERC-2.54-8P-GN" (at 83.82 102.87 0)
       (effects (font (size 1.27 1.27)) hide)
     )
@@
       (effects (font (size 1.27 1.27)) hide)
     )
+    (property "LCSC" "C2927509" (at 83.82 102.87 0)
+      (effects (font (size 1.27 1.27)) hide)
+    )
