File: hardware/EDA-Files/REG1-App-8xBE/REG1-App-8xBE.kicad_pcb (KiCad board)
At the start: 2 copper layers, 83 x 32.8 mm, 4 parts, among them J1 REG1_App_Connector, J10 Conn_01x08, J20 Conn_01x08

Commit message: wip 8xBE
Parts:
- J10, J20: footprint EasyEDALib:CONN-TH_8P-P2.54_DIBO_DB2ERC-2.54-8P-GN -> EasyEDAModLib:CONN-TH_8P-P2.54_DIBO_DB2ERC-2.54-8P-GN
Changed lines of the file:
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@@
   (net 25 "unconnected-(J20-Pin_8-Pad8)")
   (net 26 "unconnected-(J20-Pin_7-Pad7)")
-  (footprint "EasyEDALib:CONN-TH_8P-P2.54_DIBO_DB2ERC-2.54-8P-GN" (layer "F.Cu")
+  (footprint "EasyEDAModLib:CONN-TH_8P-P2.54_DIBO_DB2ERC-2.54-8P-GN" (layer "F.Cu")
     (at 76.5 106.99 -90)
     (descr "CONN-TH_8P-P2.54_DIBO_DB2ERC-2.54-8P-GN footprint")
-    (tags "CONN-TH_8P-P2.54_DIBO_DB2ERC-2.54-8P-GN footprint")
+    (tags "CONN-TH_8P-P2.54_DIBO_DB2ERC-2.54-8P-GN footprint C2927509")
     (property "LCSC" "C2927509")
     (property "Sheetfile" "REG1-App-8xBE.kicad_sch")
@@
         (effects (font (size 1 1) (thickness 0.15)))
     )
-    (fp_text value "Conn_01x08" (at 0 10.9 -90) (layer "F.Fab")
+    (fp_text value "Conn_01x08" (at 0 10.9 -90) (layer "F.Fab") hide
         (effects (font (size 1 1) (thickness 0.15)))
     )
@@
     )
     (fp_line (start -11.090018 -1.2) (end -10.003251 -1.2)
-      (stroke (width 0.254001) (type solid)) (layer "F.SilkS"))
+      (stroke (width 0.254) (type solid)) (layer "F.SilkS"))
     (fp_line (start -11.090018 8.9) (end -11.090018 -1.2)
-      (stroke (width 0.254001) (type solid)) (layer "F.SilkS"))
+      (stroke (width 0.254) (type solid)) (layer "F.SilkS"))
     (fp_line (start -11.090018 8.9) (end 11.090018 8.9)
-      (stroke (width 0.254001) (type solid)) (layer "F.SilkS"))
+      (stroke (width 0.254) (type solid)) (layer "F.SilkS"))
     (fp_line (start -7.776784 -1.2) (end -6.616104 -1.2)
-      (stroke (width 0.254001) (type solid)) (layer "F.SilkS"))
+      (stroke (width 0.254) (type solid)) (layer "F.SilkS"))
     (fp_line (start -6.083922 -1.2) (end -4.076099 -1.2)
-      (stroke (width 0.254001) (type solid)) (layer "F.SilkS"))
+      (stroke (width 0.254) (type solid)) (layer "F.SilkS"))
     (fp_line (start -3.543917 -1.2) (end -1.536093 -1.2)
-      (stroke (width 0.254001) (type solid)) (layer "F.SilkS"))
+      (stroke (width 0.254) (type solid)) (layer "F.SilkS"))
     (fp_line (start -1.003912 -1.2) (end 1.003912 -1.2)
-      (stroke (width 0.254001) (type solid)) (layer "F.SilkS"))
+      (stroke (width 0.254) (type solid)) (layer "F.SilkS"))
     (fp_line (start 1.536093 -1.2) (end 3.543917 -1.2)
-      (stroke (width 0.254001) (type solid)) (layer "F.SilkS"))
+      (stroke (width 0.254) (type solid)) (layer "F.SilkS"))
     (fp_line (start 4.076099 -1.2) (end 6.083922 -1.2)
-      (stroke (width 0.254001) (type solid)) (layer "F.SilkS"))
+      (stroke (width 0.254) (type solid)) (layer "F.SilkS"))
     (fp_line (start 6.616104 -1.2) (end 8.623927 -1.2)
-      (stroke (width 0.254001) (type solid)) (layer "F.SilkS"))
+      (stroke (width 0.254) (type solid)) (layer "F.SilkS"))
     (fp_line (start 9.156109 -1.2) (end 11.090018 -1.2)
-      (stroke (width 0.254001) (type solid)) (layer "F.SilkS"))
+      (stroke (width 0.254) (type solid)) (layer "F.SilkS"))
     (fp_line (start 11.090018 8.9) (end 11.090018 -1.2)
-      (stroke (width 0.254001) (type solid)) (layer "F.SilkS"))
+      (stroke (width 0.254) (type solid)) (layer "F.SilkS"))
+    (fp_line (start -11.3 -1.4) (end 11.3 -1.4)
+      (stroke (width 0.05) (type default)) (layer "F.CrtYd"))
+    (fp_line (start -11.3 9.1) (end -11.3 -1.4)
+      (stroke (width 0.05) (type default)) (layer "F.CrtYd"))
+    (fp_line (start 11.3 -1.4) (end 11.3 9.1)
+      (stroke (width 0.05) (type default)) (layer "F.CrtYd"))
+    (fp_line (start 11.3 9.1) (end -11.3 9.1)
+      (stroke (width 0.05) (type default)) (layer "F.CrtYd"))
     (pad "1" thru_hole rect (at -8.890018 0 270) (size 2 2) (drill 1.4) (layers "*.Cu" "*.Mask")
       (net 11 "unconnected-(J10-Pin_1-Pad1)") (pinfunction "Pin_1") (pintype "passive"))
@@
       (net 23 "unconnected-(J10-Pin_8-Pad8)") (pinfunction "Pin_8") (pintype "passive"))
     (model "${EASYEDALIB_DIR}/EasyEDALib.3dshapes/CONN-TH_8P-P2.54_DIBO_DB2ERC-2.54-8P-GN.step"
-      (offset (xyz 0 0 0))
+      (offset (xyz 0 -3.8 0))
       (scale (xyz 1 1 1))
       (rotate (xyz 0 0 0))
     )
   )
-  (footprint "EasyEDALib:CONN-TH_8P-P2.54_DIBO_DB2ERC-2.54-8P-GN" (layer "F.Cu")
+  (footprint "EasyEDAModLib:CONN-TH_8P-P2.54_DIBO_DB2ERC-2.54-8P-GN" (layer "F.Cu")
     (at 146.53 106.99 90)
     (descr "CONN-TH_8P-P2.54_DIBO_DB2ERC-2.54-8P-GN footprint")
-    (tags "CONN-TH_8P-P2.54_DIBO_DB2ERC-2.54-8P-GN footprint")
+    (tags "CONN-TH_8P-P2.54_DIBO_DB2ERC-2.54-8P-GN footprint C2927509")
     (property "LCSC" "C2927509")
     (property "Sheetfile" "REG1-App-8xBE.kicad_sch")
@@
         (effects (font (size 1 1) (thickness 0.15)))
     )
-    (fp_text value "Conn_01x08" (at 0 10.9 90) (layer "F.Fab")
+    (fp_text value "Conn_01x08" (at 0 10.9 90) (layer "F.Fab") hide
         (effects (font (size 1 1) (thickness 0.15)))
     )
@@
     )
     (fp_line (start -11.090018 -1.2) (end -10.003251 -1.2)
-      (stroke (width 0.254001) (type solid)) (layer "F.SilkS"))
+      (stroke (width 0.254) (type solid)) (layer "F.SilkS"))
     (fp_line (start -11.090018 8.9) (end -11.090018 -1.2)
-      (stroke (width 0.254001) (type solid)) (layer "F.SilkS"))
+      (stroke (width 0.254) (type solid)) (layer "F.SilkS"))
     (fp_line (start -11.090018 8.9) (end 11.090018 8.9)
-      (stroke (width 0.254001) (type solid)) (layer "F.SilkS"))
+      (stroke (width 0.254) (type solid)) (layer "F.SilkS"))
     (fp_line (start -7.776784 -1.2) (end -6.616104 -1.2)
-      (stroke (width 0.254001) (type solid)) (layer "F.SilkS"))
+      (stroke (width 0.254) (type solid)) (layer "F.SilkS"))
     (fp_line (start -6.083922 -1.2) (end -4.076099 -1.2)
-      (stroke (width 0.254001) (type solid)) (layer "F.SilkS"))
+      (stroke (width 0.254) (type solid)) (layer "F.SilkS"))
     (fp_line (start -3.543917 -1.2) (end -1.536093 -1.2)
-      (stroke (width 0.254001) (type solid)) (layer "F.SilkS"))
+      (stroke (width 0.254) (type solid)) (layer "F.SilkS"))
     (fp_line (start -1.003912 -1.2) (end 1.003912 -1.2)
-      (stroke (width 0.254001) (type solid)) (layer "F.SilkS"))
+      (stroke (width 0.254) (type solid)) (layer "F.SilkS"))
     (fp_line (start 1.536093 -1.2) (end 3.543917 -1.2)
-      (stroke (width 0.254001) (type solid)) (layer "F.SilkS"))
+      (stroke (width 0.254) (type solid)) (layer "F.SilkS"))
     (fp_line (start 4.076099 -1.2) (end 6.083922 -1.2)
-      (stroke (width 0.254001) (type solid)) (layer "F.SilkS"))
+      (stroke (width 0.254) (type solid)) (layer "F.SilkS"))
     (fp_line (start 6.616104 -1.2) (end 8.623927 -1.2)
-      (stroke (width 0.254001) (type solid)) (layer "F.SilkS"))
+      (stroke (width 0.254) (type solid)) (layer "F.SilkS"))
     (fp_line (start 9.156109 -1.2) (end 11.090018 -1.2)
-      (stroke (width 0.254001) (type solid)) (layer "F.SilkS"))
+      (stroke (width 0.254) (type solid)) (layer "F.SilkS"))
     (fp_line (start 11.090018 8.9) (end 11.090018 -1.2)
-      (stroke (width 0.254001) (type solid)) (layer "F.SilkS"))
+      (stroke (width 0.254) (type solid)) (layer "F.SilkS"))
+    (fp_line (start -11.3 -1.4) (end 11.3 -1.4)
+      (stroke (width 0.05) (type default)) (layer "F.CrtYd"))
+    (fp_line (start -11.3 9.1) (end -11.3 -1.4)
+      (stroke (width 0.05) (type default)) (layer "F.CrtYd"))
+    (fp_line (start 11.3 -1.4) (end 11.3 9.1)
+      (stroke (width 0.05) (type default)) (layer "F.CrtYd"))
+    (fp_line (start 11.3 9.1) (end -11.3 9.1)
+      (stroke (width 0.05) (type default)) (layer "F.CrtYd"))
     (pad "1" thru_hole rect (at -8.890018 0 90) (size 2 2) (drill 1.4) (layers "*.Cu" "*.Mask")
       (net 17 "unconnected-(J20-Pin_1-Pad1)") (pinfunction "Pin_1") (pintype "passive"))
@@
       (net 25 "unconnected-(J20-Pin_8-Pad8)") (pinfunction "Pin_8") (pintype "passive"))
     (model "${EASYEDALIB_DIR}/EasyEDALib.3dshapes/CONN-TH_8P-P2.54_DIBO_DB2ERC-2.54-8P-GN.step"
-      (offset (xyz 0 0 0))
+      (offset (xyz 0 -3.8 0))
       (scale (xyz 1 1 1))
       (rotate (xyz 0 0 0))
