File: hardware/EDA-Files/REG1-App-Dali/REG1-App-Dali.kicad_sch (KiCad schematic)
At the start: 26 parts, among them J1 REG1_App_Connector, J2 Dali, Q1 BSS123, Q2 BC857, U1 EL817S1(C)(TU)-F, U2 EL817S1(C)(TU)-F, U3 STN93003, U4 STN1HNK60

Commit message: add wip for a dali power supply
Parts:
- removed D4: LED, LED_SMD:LED_0603_1608Metric, symbol Device:LED
- removed R11: 300, Resistor_SMD:R_1206_3216Metric, symbol Device:R
- removed R8: 4.7k, Resistor_SMD:R_0603_1608Metric, symbol Device:R
Connections:
- net D_TX: now also R10.2
Other:
- added sheet Dali Power Supply (dali_power_supply.kicad_sch)
- moved on the sheet: R9
Changed lines of the file:
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@@
   (junction (at 109.855 140.97) (diameter 0) (color 0 0 0 0)
   )
-  (junction (at 271.78 17.78) (diameter 0) (color 0 0 0 0)
-  )
   (junction (at 97.79 123.19) (diameter 0) (color 0 0 0 0)
   )
@@
   (junction (at 152.4 105.41) (diameter 0) (color 0 0 0 0)
   )
-  (junction (at 233.68 25.4) (diameter 0) (color 0 0 0 0)
-  )
   (junction (at 78.74 123.19) (diameter 0) (color 0 0 0 0)
   )
@@
     (stroke (width 0) (type default))
   )
-  (wire (pts (xy 261.62 25.4) (xy 271.78 25.4))
-    (stroke (width 0) (type default))
-  )
   (wire (pts (xy 81.28 34.29) (xy 86.36 34.29))
     (stroke (width 0) (type default))
@@
     (stroke (width 0) (type default))
   )
-  (wire (pts (xy 271.78 25.4) (xy 271.78 17.78))
-    (stroke (width 0) (type default))
-  )
   (wire (pts (xy 181.61 125.73) (xy 181.61 140.97))
     (stroke (width 0) (type default))
   )
-  (wire (pts (xy 233.68 25.4) (xy 238.76 25.4))
-    (stroke (width 0) (type default))
-  )
   (wire (pts (xy 137.16 140.97) (xy 123.19 140.97))
     (stroke (width 0) (type default))
@@
     (stroke (width 0) (type default))
   )
-  (wire (pts (xy 256.54 17.78) (xy 271.78 17.78))
+  (wire (pts (xy 255.27 25.4) (xy 270.51 25.4))
     (stroke (width 0) (type default))
   )
@@
     (stroke (width 0) (type default))
   )
-  (wire (pts (xy 261.62 58.42) (xy 256.54 58.42))
-    (stroke (width 0) (type default))
-  )
   (wire (pts (xy 30.48 82.55) (xy 30.48 80.01))
     (stroke (width 0) (type default))
@@
     (stroke (width 0) (type default))
   )
-  (wire (pts (xy 233.68 17.78) (xy 233.68 25.4))
-    (stroke (width 0) (type default))
-  )
   (wire (pts (xy 170.18 124.46) (xy 170.18 140.97))
     (stroke (width 0) (type default))
@@
     (stroke (width 0) (type default))
   )
+  (wire (pts (xy 228.6 25.4) (xy 247.65 25.4))
+    (stroke (width 0) (type default))
+  )
   (wire (pts (xy 228.6 30.48) (xy 231.14 30.48))
     (stroke (width 0) (type default))
@@
     (stroke (width 0) (type default))
   )
-  (wire (pts (xy 246.38 25.4) (xy 254 25.4))
-    (stroke (width 0) (type default))
-  )
-  (wire (pts (xy 248.92 17.78) (xy 233.68 17.78))
-    (stroke (width 0) (type default))
-  )
   (wire (pts (xy 109.855 80.01) (xy 109.855 100.33))
     (stroke (width 0) (type default))
@@
     (stroke (width 0) (type default))
   )
-  (wire (pts (xy 245.11 58.42) (xy 248.92 58.42))
+  (wire (pts (xy 245.11 58.42) (xy 261.62 58.42))
     (stroke (width 0) (type default))
   )
@@
   )
   (wire (pts (xy 181.61 30.48) (xy 181.61 58.42))
-    (stroke (width 0) (type default))
-  )
-  (wire (pts (xy 228.6 25.4) (xy 233.68 25.4))
     (stroke (width 0) (type default))
   )
@@
     (effects (font (size 1.27 1.27)) (justify left bottom))
   )
-  (label "D_RX" (at 234.95 17.78 0) (fields_autoplaced)
+  (label "D_RX" (at 233.68 25.4 0) (fields_autoplaced)
     (effects (font (size 1.27 1.27)) (justify left bottom))
   )
@@
     )
   )
-  (symbol (lib_id "Device:R") (at 252.73 17.78 270) (unit 1)
-    (in_bom yes) (on_board yes) (dnp no) (fields_autoplaced)
-    (property "Reference" "R9" (at 252.73 12.7 90)
-      (effects (font (size 1.27 1.27)))
-    )
-    (property "Value" "4.7k" (at 252.73 15.24 90)
-      (effects (font (size 1.27 1.27)))
-    )
-    (property "Footprint" "Resistor_SMD:R_0603_1608Metric" (at 252.73 16.002 90)
-      (effects (font (size 1.27 1.27)) hide)
-    )
-    (property "Datasheet" "~" (at 252.73 17.78 0)
-      (effects (font (size 1.27 1.27)) hide)
-    )
-    (property "LCSC" "C23162" (at 252.73 17.78 0)
+  (symbol (lib_id "Device:R") (at 251.46 25.4 270) (unit 1)
+    (in_bom yes) (on_board yes) (dnp no) (fields_autoplaced)
+    (property "Reference" "R9" (at 251.46 20.32 90)
+      (effects (font (size 1.27 1.27)))
+    )
+    (property "Value" "4.7k" (at 251.46 22.86 90)
+      (effects (font (size 1.27 1.27)))
+    )
+    (property "Footprint" "Resistor_SMD:R_0603_1608Metric" (at 251.46 23.622 90)
+      (effects (font (size 1.27 1.27)) hide)
+    )
+    (property "Datasheet" "~" (at 251.46 25.4 0)
+      (effects (font (size 1.27 1.27)) hide)
+    )
+    (property "LCSC" "C23162" (at 251.46 25.4 0)
       (effects (font (size 1.27 1.27)) hide)
     )
@@
         (path "/a0393b09-4b2d-4a64-98b7-96bb7f245f9d"
           (reference "R9") (unit 1)
-        )
-      )
-    )
-  )
-  (symbol (lib_id "Device:LED") (at 257.81 25.4 0) (unit 1)
-    (in_bom yes) (on_board yes) (dnp no) (fields_autoplaced)
-    (property "Reference" "D4" (at 256.2225 20.32 0)
-      (effects (font (size 1.27 1.27)))
-    )
-    (property "Value" "LED" (at 256.2225 22.86 0)
-      (effects (font (size 1.27 1.27)))
-    )
-    (property "Footprint" "LED_SMD:LED_0603_1608Metric" (at 257.81 25.4 0)
-      (effects (font (size 1.27 1.27)) hide)
-    )
-    (property "Datasheet" "~" (at 257.81 25.4 0)
-      (effects (font (size 1.27 1.27)) hide)
-    )
-    (property "LCSC" "C2290" (at 257.81 25.4 0)
-      (effects (font (size 1.27 1.27)) hide)
-    )
-    (pin "1")
-    (pin "2")
-    (instances
-      (project "REG1-App-Dali"
-        (path "/a0393b09-4b2d-4a64-98b7-96bb7f245f9d"
-          (reference "D4") (unit 1)
         )
       )
@@
     )
   )
-  (symbol (lib_id "Device:R") (at 242.57 25.4 270) (unit 1)
-    (in_bom yes) (on_board yes) (dnp no) (fields_autoplaced)
-    (property "Reference" "R8" (at 242.57 20.32 90)
-      (effects (font (size 1.27 1.27)))
-    )
-    (property "Value" "4.7k" (at 242.57 22.86 90)
-      (effects (font (size 1.27 1.27)))
-    )
-    (property "Footprint" "Resistor_SMD:R_0603_1608Metric" (at 242.57 23.622 90)
-      (effects (font (size 1.27 1.27)) hide)
-    )
-    (property "Datasheet" "~" (at 242.57 25.4 0)
-      (effects (font (size 1.27 1.27)) hide)
-    )
-    (property "LCSC" "C23162" (at 242.57 25.4 0)
-      (effects (font (size 1.27 1.27)) hide)
-    )
-    (pin "1")
-    (pin "2")
-    (instances
-      (project "REG1-App-Dali"
-        (path "/a0393b09-4b2d-4a64-98b7-96bb7f245f9d"
-          (reference "R8") (unit 1)
-        )
-      )
-    )
-  )
   (symbol (lib_id "DALI:EL357N(A)(TA)-G") (at 215.9 60.96 0) (mirror y) (unit 1)
     (in_bom yes) (on_board yes) (dnp no)
@@
     )
   )
-  (symbol (lib_id "Device:R") (at 252.73 58.42 90) (unit 1)
-    (in_bom yes) (on_board yes) (dnp no) (fields_autoplaced)
-    (property "Reference" "R11" (at 252.73 53.34 90)
-      (effects (font (size 1.27 1.27)))
-    )
-    (property "Value" "300" (at 252.73 55.88 90)
-      (effects (font (size 1.27 1.27)))
-    )
-    (property "Footprint" "Resistor_SMD:R_1206_3216Metric" (at 252.73 60.198 90)
-      (effects (font (size 1.27 1.27)) hide)
-    )
-    (property "Datasheet" "~" (at 252.73 58.42 0)
-      (effects (font (size 1.27 1.27)) hide)
-    )
-    (property "LCSC" "C17887" (at 252.73 58.42 0)
-      (effects (font (size 1.27 1.27)) hide)
-    )
-    (pin "1")
-    (pin "2")
-    (instances
-      (project "REG1-App-Dali"
-        (path "/a0393b09-4b2d-4a64-98b7-96bb7f245f9d"
-          (reference "R11") (unit 1)
-        )
-      )
-    )
-  )
   (symbol (lib_id "DALI:BSS123") (at 123.19 120.65 0) (unit 1)
     (in_bom yes) (on_board yes) (dnp no) (fields_autoplaced)
@@
     )
   )
-  (symbol (lib_id "power:+3.3V") (at 271.78 17.78 0) (unit 1)
-    (in_bom yes) (on_board yes) (dnp no) (fields_autoplaced)
-    (property "Reference" "#PWR02" (at 271.78 21.59 0)
-      (effects (font (size 1.27 1.27)) hide)
-    )
-    (property "Value" "+3.3V" (at 271.78 13.97 0)
-      (effects (font (size 1.27 1.27)))
-    )
-    (property "Footprint" "" (at 271.78 17.78 0)
-      (effects (font (size 1.27 1.27)) hide)
-    )
-    (property "Datasheet" "" (at 271.78 17.78 0)
+  (symbol (lib_id "power:+3.3V") (at 270.51 25.4 0) (unit 1)
+    (in_bom yes) (on_board yes) (dnp no) (fields_autoplaced)
+    (property "Reference" "#PWR02" (at 270.51 29.21 0)
+      (effects (font (size 1.27 1.27)) hide)
+    )
+    (property "Value" "+3.3V" (at 270.51 21.59 0)
+      (effects (font (size 1.27 1.27)))
+    )
+    (property "Footprint" "" (at 270.51 25.4 0)
+      (effects (font (size 1.27 1.27)) hide)
+    )
+    (property "Datasheet" "" (at 270.51 25.4 0)
       (effects (font (size 1.27 1.27)) hide)
     )
@@
       )
     )
+  )
+  (sheet (at 16.51 17.78) (size 25.4 10.16) (fields_autoplaced)
+    (stroke (width 0.1524) (type solid))
+    (fill (color 0 0 0 0.0000))
+    (property "Sheetname" "Dali Power Supply" (at 16.51 17.0684 0)
+      (effects (font (size 1.27 1.27)) (justify left bottom))
+    )
+    (property "Sheetfile" "dali_power_supply.kicad_sch" (at 16.51 28.5246 0)
+      (effects (font (size 1.27 1.27)) (justify left top))
+    )
+    (instances
+      (project "REG1-App-Dali"
+        (path "/a0393b09-4b2d-4a64-98b7-96bb7f245f9d" (page "2"))
+      )
+    )
