File: hardware/EDA-Files/REG1-App-GW-RF2G4/REG1-App-GW-RF2G4.kicad_pcb (KiCad board)
At the start: 2 copper layers, 83 x 32.8 mm, 5 parts, among them J1 REG1_App_Connector, U1 E01-ML01DP5, U2 E01-2G4M27S, U3 E07-M1101D-TH

Commit message: wip GW RF
Parts:
- removed the G*** at (138.9, 95.8)
- removed U3: E07-M1101D-TH, EasyEDALib:WIRELM-TH_E07-M1101D-TH
- added G***: LOGO, OpenKNX:OpenKNX_Logo_10x10, F.Cu at (139.4, 114.8)
- added G1: LOGO, OpenKNX:CC-BY-NY-SA_12x4, F.Cu at (141.3, 119.9)
Routing:
- net CS: track 71.8 -> 34.3 mm
- net MOSI: track 68.3 -> 35.7 mm
- net INT: track 56.0 -> 33.5 mm, vias 1 -> 0
- net +3.3V: track 60.9 -> 39.0 mm, vias 1 -> 0
- net GND: track 81.0 -> 60.2 mm, vias 2 -> 1
- net MISO: track 78.9 -> 60.3 mm, vias 2 -> 1
- net CLK: track 68.7 -> 55.6 mm, vias 2 -> 1
- net enable: track 63.0 -> 54.7 mm
Other:
- board text added: "REG1-App-GW-RF2G4 V00.01 (c) Ing-Dom, 2024"
- board text removed: "REG1-App-RF01 V00.01 (c) Ing-Dom, 2024"

Commit message: App-GW-RF2G4 V00.01
Parts:
- moved G*** 28.8 mm to (113.5, 102.3)
- moved G1 24.6 mm to (124.0, 102.3)
Connections:
- J1 pad 1: enable -> unconnected-(J1-GP16-Pad1)
- J1 pad 2: unconnected-(J1-GP17-Pad2) -> enable
Routing:
- net enable: track 54.7 -> 52.2 mm
Other:
- board text added: "REG1-App-GW-RF2G4 V00.01 by Ing-Dom, 2024"
- board text removed: "REG1-App-GW-RF2G4 V00.01 (c) Ing-Dom, 2024"
Changed lines of the file:
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@@
   (paper "A4")
   (title_block
-    (date "2024-07-27")
-    (rev "V01.00")
+    (date "2024-07-29")
+    (rev "V00.01")
   )
   (layers
@@
   )
   (net 0 "")
-  (net 1 "unconnected-(J1-GP17-Pad2)")
+  (net 1 "unconnected-(J1-GP16-Pad1)")
   (net 2 "unconnected-(J1-VCC2-Pad10)")
   (net 3 "unconnected-(U1-Pad12)")
@@
   )
   (footprint "OpenKNX:CC-BY-NY-SA_12x4" (layer "F.Cu")
-    (at 141.325111 119.895111)
+    (at 124.05 102.35)
     (attr board_only exclude_from_pos_files exclude_from_bom)
     (fp_text reference "G1" (at 0 0) (layer "F.Fab")
@@
   )
   (footprint "OpenKNX:OpenKNX_Logo_10x10" (layer "F.Cu")
-    (at 139.42 114.81)
+    (at 113.5 102.35)
     (attr board_only exclude_from_pos_files exclude_from_bom)
     (fp_text reference "G***" (at 0 0) (layer "F.Fab")
@@
       (stroke (width 0.1) (type solid)) (layer "B.Fab"))
     (pad "1" thru_hole rect locked (at 0 0 90) (size 1.7 1.7) (drill 1) (layers "*.Cu" "*.Mask")
-      (net 7 "enable") (pinfunction "GP16") (pintype "bidirectional"))
+      (net 1 "unconnected-(J1-GP16-Pad1)") (pinfunction "GP16") (pintype "bidirectional"))
     (pad "2" thru_hole oval locked (at 0 -2.54 90) (size 1.7 1.7) (drill 1) (layers "*.Cu" "*.Mask")
-      (net 1 "unconnected-(J1-GP17-Pad2)") (pinfunction "GP17") (pintype "bidirectional"))
+      (net 7 "enable") (pinfunction "GP17") (pintype "bidirectional"))
     (pad "3" thru_hole oval locked (at 0 -5.08 90) (size 1.7 1.7) (drill 1) (layers "*.Cu" "*.Mask")
       (net 8 "INT") (pinfunction "GP18") (pintype "bidirectional"))
@@
   (gr_line (start 140.9 90.1) (end 140.9 92.4)
     (stroke (width 0.05) (type solid)) (layer "Edge.Cuts"))
-  (gr_text "REG1-App-GW-RF2G4 V00.01\n(c) Ing-Dom, 2024" (at 81.95 94.9) (layer "F.SilkS")
+  (gr_text "REG1-App-GW-RF2G4 V00.01\nby Ing-Dom, 2024" (at 109.85 98) (layer "F.SilkS")
     (effects (font (size 1 1) (thickness 0.15)) (justify left))
   )
@@
     (effects (font (size 1 1) (thickness 0.15)) (justify left bottom))
   )
-  (segment (start 116.833503 101.933503) (end 110.1 108.667007) (width 0.3) (layer "F.Cu") (net 7))
-  (segment (start 127.21 97.85) (end 120.917007 97.85) (width 0.3) (layer "F.Cu") (net 7))
-  (segment (start 120.917007 97.85) (end 116.833503 101.933503) (width 0.3) (layer "F.Cu") (net 7))
+  (segment (start 120.917007 97.85) (end 124.67 97.85) (width 0.3) (layer "F.Cu") (net 7))
+  (segment (start 110.1 108.667007) (end 120.917007 97.85) (width 0.3) (layer "F.Cu") (net 7))
   (segment (start 97.55 110.68) (end 95.63 110.68) (width 0.3) (layer "F.Cu") (net 7))
   (segment (start 95.63 110.68) (end 95.6 110.65) (width 0.3) (layer "F.Cu") (net 7))
-  (segment (start 130.76 94.3) (end 127.21 97.85) (width 0.3) (layer "F.Cu") (net 7))
+  (segment (start 124.67 97.85) (end 128.22 94.3) (width 0.3) (layer "F.Cu") (net 7))
   (segment (start 103.790043 108.667007) (end 110.1 108.667007) (width 0.3) (layer "F.Cu") (net 7))
   (via (at 95.6 110.65) (size 0.6) (drill 0.3) (layers "F.Cu" "B.Cu") (net 7))
