File: hardware/EDA-Files/REG1-App-SEN-Multi/REG1-App-SEN-Multi.kicad_pcb (KiCad board)
At the start: 2 copper layers, 83 x 32.8 mm, 26 parts, among them J1 REG1_App_Connector, J10 RJ22_1, J11 RJ22_2, J13 Conn_01x08, J20 Conn_01x06, U10 USBLC6-2SC6, U11 USBLC6-2SC6, U20 CA-IS3644

Commit message: REG1-App-SEN-Multi V01.00 - editorial change to V01.00 after Beta
Parts:
- added REF**: JLCPCB_Tooling_hole, DomsKiCADLib:JLCPCB_Tooling_hole, F.Cu at (71.5, 117.2)
- added REF**: JLCPCB_Tooling_hole, DomsKiCADLib:JLCPCB_Tooling_hole, F.Cu at (139.2, 91.8)
- J10: value RJ22_1 -> RJ22
- J11: value RJ22_2 -> RJ22
Other:
- board text added: "REG1-App-SEN-Multi V01.00 by Ing-Dom, 2026"
- board text removed: "REG1-App-SEN-Multi V00.02 by Ing-Dom, 2024"
