File: hardware/EDA-Files/REG1-App-SEN-Multi/REG1-App-SEN-Multi.kicad_sch (KiCad schematic)
At the start: 24 parts, among them J1 REG1_App_Connector, J10 RJ22_1, J11 RJ22_2, J13 Conn_01x08, J20 Conn_01x06, U10 USBLC6-2SC6, U11 USBLC6-2SC6, U20 CA-IS3644

Commit message: REG1-App-SEN-Multi V01.00 - editorial change to V01.00 after Beta
Parts:
- J10: value RJ22_1 -> RJ22
- J11: value RJ22_2 -> RJ22
- J13: now not fitted; now left out of the parts list
